Commit message: Update VLM-CBF PyBullet training, env, and evaluation code

File: assets/base_diff.urdf (robot description, URDF)
Before this commit: robot base_diff, 3 links, 2 joints
Links:
- link wheel_left: mass None -> 1.0
- link wheel_right: mass None -> 1.0

File: assets/base_omni.urdf (robot description, URDF)
Before this commit: robot base_omni, 5 links, 4 joints
Links:
- link wheel_fl: mass None -> 1.0
- link wheel_fr: mass None -> 1.0
- link wheel_rl: mass None -> 1.0
- link wheel_rr: mass None -> 1.0
